Commit message: Fixed tum_simulator to compile with gazebo-7.0.0 and ros kinetic kame. diffdrive_plugin_6w needs another look, since physics behavior was changed in gazebo.

File: cvg_sim_gazebo/urdf/quadrotor.urdf.xacro (robot description, xacro)
@@ -4,5 +4,5 @@
     xmlns:controller="http://playerstage.sourceforge.net/gazebo/xmlschema/#controller"
     xmlns:interface="http://playerstage.sourceforge.net/gazebo/xmlschema/#interface"
-    xmlns:xacro="http://playerstage.sourceforge.net/gazebo/xmlschema/#interface">
+    xmlns:xacro="http://ros.org/wiki/xacro">
     <!-- Included URDF Files -->
     <xacro:include filename="$(find cvg_sim_gazebo)/urdf/quadrotor_base.urdf.xacro" />

File: cvg_sim_gazebo/urdf/quadrotor_base.urdf.xacro (robot description, xacro)
@@ -9,4 +9,5 @@
   <!-- Main quadrotor link -->
   <xacro:macro name="quadrotor_base_macro">
+	<link name="dummy_root"/>
     <link name="base_link">
       <inertial>
@@ -28,4 +29,8 @@
       </collision>
     </link>
+	<joint name="dummy_to_base" type="fixed">
+	  <parent link="dummy_root"/>
+	  <child link="base_link"/>
+	</joint>
     <gazebo reference="base_link">
       <turnGravityOff>false</turnGravityOff>

File: cvg_sim_gazebo/urdf/quadrotor_sensors.urdf.xacro (robot description, xacro)
@@ -4,6 +4,6 @@
 xmlns:controller="http://playerstage.sourceforge.net/gazebo/xmlschema/#controller"
 xmlns:interface="http://playerstage.sourceforge.net/gazebo/xmlschema/#interface"
-xmlns:xacro="http://playerstage.sourceforge.net/gazebo/xmlschema/#interface">
-    <property name="M_PI" value="3.1415926535897931" />
+xmlns:xacro="http://ros.org/wiki/xacro">
+    <xacro:property name="M_PI" value="3.1415926535897931" />
     <!-- Included URDF Files -->
     <xacro:include filename="$(find cvg_sim_gazebo)/urdf/quadrotor_base.urdf.xacro" />
@@ -27,5 +27,5 @@
     </xacro:generic_camera>
     <!-- Downward facing camera -->
-    <xacro:include filename="$(find cvg_sim_gazebo)/urdf/sensors/generic_camera.urdf.xacro" />
+<!--    <xacro:include filename="$(find cvg_sim_gazebo)/urdf/sensors/generic_camera.urdf.xacro" /> -->
     <xacro:generic_camera name="bottom" sim_name="ardrone" parent="base_link" update_rate="60" res_x="640" res_y="360" image_format="R8G8B8" hfov="${81*M_PI/180}">
       <origin xyz="0.15 0.0 0.0" rpy="0 ${M_PI/2} 0"/>

File: cvg_sim_gazebo/urdf/sensors/generic_camera.urdf.xacro (robot description, xacro)
@@ -84,5 +84,5 @@
         </plugin>
       </sensor>
-      <turnGravityOff>true</turnGravityOff>
+      <!-- <turnGravityOff>true</turnGravityOff> -->
       <material>Gazebo/Blue</material>
     </gazebo>
